Commit message: 4.1

File: envs/models/Diana7_Magnet/Diana7_Magnet_red.urdf (robot description, URDF)
Before this commit: robot diana7, 10 links, 9 joints
Links:
- link end_effector: geometry collision mesh filename=./meshes/collision/end_effector.stl; visual mesh filename=./meshes/visual/end_effector.stl
